Commit message: Finished Step 2

File: Step2/rrbot.urdf.xacro (robot description, xacro)
@@ -6,4 +6,5 @@
   <!-- create link fixed to the "world" -->
   <link name="world" />
+  <link name="table_top" />
   <!-- create the first robot -->
   <xacro:rrbot prefix="rrbot1_" parent="world">

File: Step2/rrbot_on_table.urdf.xacro (robot description, xacro)
@@ -5,8 +5,9 @@
     <xacro:include filename="rrbot_macro.xacro" />
     <link name="world" />
+    <!--link name="table_top" /-->
     <xacro:table prefix="table_" parent="world">
         <origin xyz="0 0 1" rpy="0 0 0" />
     </xacro:table>
-    <xacro:rrbot prefix="rrbot_" parent="table_top">
+   <xacro:rrbot prefix="rrbot_" parent="table_top_link">
         <origin xyz="0 0 0" rpy="0 0 0" />
     </xacro:rrbot>

File: Step2/table_macro.xacro (robot description, xacro)
@@ -1,5 +1,4 @@
 <?xml version="1.0"?>
 <robot xmlns:xacro="http://www.ros.org/wiki/xacro">
-<!-- File-level so both macros can see them -->
 <xacro:property name="table_length" value="4.0" />
 <xacro:property name="table_width" value="3.0" />
@@ -41,4 +40,10 @@
     </visual>
   </link>
+  <joint name="${prefix}top_joint" type="fixed">
+    <parent link="${prefix}base_link" />
+    <child link="${prefix}top_link" />
+    <origin xyz="0 0 ${table_height}" rpy="0 0 0" />
+  </joint>
+  <link name="${prefix}top_link" />
   <xacro:table_leg prefix="${prefix}" name="leg1" x="${leg_x}"  y="${leg_y}" />
   <xacro:table_leg prefix="${prefix}" name="leg2" x="${-leg_x}" y="${leg_y}" />

File: Step2/table_on_rrbot.urdf.xacro (robot description, xacro)
@@ -9,5 +9,5 @@
     </xacro:rrbot>
     <xacro:table prefix="table_" parent="rrbot_tool0">
-        <origin xyz="0 0 0" rpy="${pi} 0 0" />
+        <origin xyz="0 0 ${table_height}" rpy="${pi} 0 0" />
     </xacro:table>
 </robot>
